File: PCB Files/Macro Pad.kicad_sch (KiCad schematic)
At the start: 30 parts, among them J1 USB_C_Receptacle_USB2.0, J2 OLED, J3 Reset, U1 ATMEGA32U4-AUR

Commit message: Adding changes
Other:
- title: (none) -> MacroPad
Changed lines of the file:
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@@
 (kicad_sch (version 20230121) (generator eeschema)
   (paper "A4")
+  (title_block
+    (title "MacroPad")
+    (date "2024-01-07")
+    (rev "3.0")
+  )
   (junction (at 27.94 34.29) (diameter 0) (color 0 0 0 0)
   )
